File: PCB/LTX-Rapidfire.brd (EAGLE design)
At the start: 52.7 x 25.1 mm, 52 parts, among them J1 F-1X08-SIP-100-40Y, Q1 MMBT3904, Q10 SS8550D, Q11 2N3906, Q12 2N3906, Q13 MMBT3904, Q2 2N3906, Q3 MMBT3904, Q4 MMBT3904, Q5 MMBT3904, Q6 2N3906, Q7 2N3906, Q8 2N3906, Q9 MMBT3904, SW1 F-1X02-SIP-100-40, U1 XC6206P332MR, U3 ATTINY1616-MNRVQFN20_3X3_MCH-M

Commit message: Updated gerbers, com, and placement
Parts:
- removed R28: 1K, SparkFun-Resistors:0402
- added R26: 1k, JLC PCB Basic Parts_loc:R0603
Connections:
- net PROGRAM_RESET_PA0: now also R26.1; no longer R28.1
- net UPDI: now also R26.2; no longer R28.2
Routing:
- net PROGRAM_RESET_PA0: track 31.3 -> 30.6 mm
Changed lines of the file:
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@@
 <setting verticaltext="up"/>
 </settings>
-<grid distance="0.05" unitdist="inch" unit="inch" style="lines" multiple="1" display="yes" altdistance="0.005" altunitdist="inch" altunit="inch"/>
+<grid distance="1" unitdist="mm" unit="mm" style="lines" multiple="1" display="yes" altdistance="0.1" altunitdist="mm" altunit="mm"/>
 <layers>
 <layer number="1" name="Top" color="4" fill="1" visible="yes" active="yes"/>
@@
 <attribute name="LCSC_PART" value="C66801" x="2.413" y="15.113" size="1.016" layer="27" font="vector" rot="R90" display="off"/>
 </element>
-<element name="R28" library="SparkFun-Resistors" package="0402" value="1K" x="2.286" y="9.34539375" rot="R225">
-<attribute name="PROD_ID" value="RES-14341" x="22.0425625" y="-6.819065625" size="1.778" layer="27" font="vector" ratio="15" rot="R225" display="off"/>
-</element>
 <element name="U3" library="attiny1616" package="VQFN20_3X3_MCH-M" value="ATTINY1616-MNRVQFN20_3X3_MCH-M" x="6.223" y="7.62" smashed="yes" rot="R45">
 <attribute name="DIGI-KEY_PART_NUMBER_1" value="ATTINY1616-MNRCT-ND" x="11.611153125" y="2.23184375" size="1.778" layer="27" font="vector" ratio="15" rot="R45" display="off"/>
@@
 </element>
 <element name="JP1" library="adafruit" package="1X03" value="" x="9.525" y="2.794"/>
+<element name="R26" library="JLC PCB Basic Parts_loc" package="R0603" value="1k" x="2.28786875" y="9.16360625" rot="R225">
+<attribute name="LCSC_PART" value="C21190" x="2.28786875" y="9.16360625" size="1.778" layer="27" font="vector" ratio="15" rot="R225" display="off"/>
+<attribute name="LCSC_ROTATION_CCW" value="0" x="2.28786875" y="9.16360625" size="1.778" layer="27" font="vector" ratio="15" rot="R225" display="off"/>
+<attribute name="LCSC_PRICE1_EUR" value="" x="2.28786875" y="9.16360625" size="1.778" layer="27" font="vector" ratio="15" rot="R225" display="off"/>
+<attribute name="LCSC_DATASHEET" value="https://datasheet.lcsc.com/lcsc/2110252030_UNI-ROYAL-Uniroyal-Elec-0603WAF1001T5E_C21190.pdf" x="2.28786875" y="9.16360625" size="1.778" layer="27" font="vector" ratio="15" rot="R225" display="off"/>
+<attribute name="LCSC_STOCK" value="5175299" x="2.28786875" y="9.16360625" size="1.778" layer="27" font="vector" ratio="15" rot="R225" display="off"/>
+<attribute name="PROPERTIES" value="±1% 1/10W Thick Film Resistors 75V ±100ppm -55°C~+155°C 1kOhm 0603  ROHS" x="2.28786875" y="9.16360625" size="1.778" layer="27" font="vector" ratio="15" rot="R225" display="off"/>
+</element>
 </elements>
 <signals>
@@
 <signal name="PROGRAM_RESET_PA0">
 <contactref element="R8" pad="1"/>
-<contactref element="R28" pad="1"/>
 <contactref element="U3" pad="19"/>
-<wire x1="3.048" y1="9.7536" x2="2.7432" y2="9.7536" width="0.1524" layer="1"/>
-<wire x1="2.7432" y1="9.7536" x2="2.696121875" y2="9.755515625" width="0.1524" layer="1"/>
 <wire x1="4.898446875" y1="8.378865625" x2="3.521796875" y2="9.755515625" width="0.2032" layer="1"/>
-<wire x1="3.521796875" y1="9.755515625" x2="2.696121875" y2="9.755515625" width="0.2032" layer="1"/>
-<wire x1="11.6332" y1="10.3632" x2="3.30380625" y2="10.3632" width="0.2032" layer="1"/>
-<wire x1="3.30380625" y1="10.3632" x2="2.696121875" y2="9.755515625" width="0.2032" layer="1"/>
 <wire x1="11.6332" y1="10.3632" x2="13.97" y2="12.7" width="0.2032" layer="1"/>
 <via x="13.97" y="12.7" extent="1-16" drill="0.381"/>
@@
 <wire x1="24.257" y1="10.033" x2="24.257" y2="6.897" width="0.2032" layer="1"/>
 <wire x1="24.257" y1="6.897" x2="24.55" y2="6.604" width="0.2032" layer="1"/>
+<contactref element="R26" pad="1"/>
+<wire x1="3.521796875" y1="9.755515625" x2="2.898040625" y2="9.755515625" width="0.2032" layer="1"/>
+<wire x1="2.898040625" y1="9.755515625" x2="2.888909375" y2="9.764646875" width="0.2032" layer="1"/>
+<wire x1="11.6332" y1="10.3632" x2="3.4874625" y2="10.3632" width="0.2032" layer="1"/>
+<wire x1="3.4874625" y1="10.3632" x2="2.888909375" y2="9.764646875" width="0.2032" layer="1"/>
 </signal>
 <signal name="N$17">
@@
 </signal>
 <signal name="UPDI">
-<contactref element="R28" pad="2"/>
 <via x="9.525" y="6.35" extent="1-16" drill="0.381"/>
 <wire x1="9.525" y1="6.35" x2="5.08" y2="6.35" width="0.254" layer="16"/>
 <wire x1="5.08" y1="6.35" x2="1.27" y2="10.16" width="0.254" layer="16"/>
 <via x="1.27" y="10.16" extent="1-16" drill="0.381"/>
-<wire x1="1.27" y1="10.16" x2="1.27" y2="9.54114375" width="0.254" layer="1"/>
-<wire x1="1.27" y1="9.54114375" x2="1.875875" y2="8.93526875" width="0.254" layer="1"/>
+<wire x1="1.27" y1="10.16" x2="1.27" y2="8.9793875" width="0.254" layer="1"/>
 <wire x1="9.525" y1="6.35" x2="9.525" y2="4.699" width="0.254" layer="1"/>
 <wire x1="9.525" y1="4.699" x2="11.684" y2="2.54" width="0.254" layer="1"/>
@@
 <wire x1="11.684" y1="2.54" x2="11.811" y2="2.54" width="0.254" layer="1"/>
 <wire x1="11.811" y1="2.54" x2="12.065" y2="2.794" width="0.254" layer="1"/>
+<contactref element="R26" pad="2"/>
+<wire x1="1.27" y1="8.9793875" x2="1.686825" y2="8.5625625" width="0.254" layer="1"/>
 </signal>
 <signal name="+9V">
